File: PCB/pcb_flyback/pcb_flyback.sch (KiCad schematic (older format))
At the start: 10 parts

Commit message: 1 Version PCB terminada (Se puede mejorar)
Parts:
- removed C?: C, symbol pspice:C
- removed D?: 1N4148, Diode_THT:D_DO-35_SOD27_P7.62mm_Horizontal, symbol Diode:1N4148
- removed R? (x2): R, symbol Device:R
- removed T?: Transformer_1P_1S, symbol Device:Transformer_1P_1S
- added C1, C2, C3, C4, C5, C6: C, Capacitor_SMD:CP_Elec_3x5.3, symbol Device:C
- added D1: D_Zener, Diode_THT:D_DO-35_SOD27_P2.54mm_Vertical_AnodeUp, symbol Device:D_Zener
- added D3: TL431D, Package_SO:SOIC-8_3.9x4.9mm_P1.27mm, symbol Reference_Voltage:TL431D
- added Dsnuber1, Dsnuber2: 1N4148, Diode_THT:D_DO-35_SOD27_P7.62mm_Horizontal, symbol Diode:1N4148
- added Out1, Out2: Screw_Terminal_01x02, Connector_Wire:SolderWirePad_1x02_P3.81mm_Drill0.8mm, symbol Connector:Screw_Terminal_01x02
- added R1, R10, R11, R12, R2, R3, R4, R5, R6, R7, R8, R9: R, Resistor_SMD:R_0201_0603Metric, symbol Device:R
- added TR1: TRANSF6, Transformer_SMD:Pulse_PA2777NL, symbol Transformer:TRANSF6
- added U2: PC817, Package_DIP:DIP-4_W7.62mm, symbol Isolator:PC817
- CSnuber1: renamed from C?; footprint (none) -> Capacitor_SMD:CP_Elec_3x5.3
- D2: renamed from D?; symbol Simulation_SPICE:DIODE -> pcb_flyback-rescue:DIODE-Simulation_SPICE
- RSnuber1: renamed from R?; footprint (none) -> Resistor_SMD:R_0201_0603Metric
- U1: renamed from U?; footprint (none) -> Package_DIP:DIP-16_W7.62mm_SMDSocket_SmallPads; symbol Regulator_Controller:TL494 -> pcb_flyback-rescue:TL494-Regulator_Controller
- gave numbers to parts that had none: 1
Connections:
- net GND: now also U1.1 (1IN+), U1.2 (1IN-), U1.4 (DTC), U1.7 (GND), C1.1, C2.2, C6.1, D1.2 (A), D3.2 (A), D3.3 (A), D3.6 (A), D3.7 (A), Out1.1 (Pin_1), R1.2, R12.2, R4.2, R7.2, TR1.4
- net at Q1.1 (G): now also U1.11 (C2), U1.8 (C1), R6.2
- net at Q1.2 (D): now also Dsnuber1.2 (A), TR1.2
- net at CSnuber1.2, RSnuber1.2: now also Dsnuber1.1 (K)
- net at CSnuber1.1, RSnuber1.1: now also Out1.2 (Pin_2), TR1.1
- net at D2.1 (A): now also TR1.8
- net at D2.2 (K): now also C5.1, Out2.1 (Pin_1), R11.1, R9.1
- net at U1.12 (VCC): now also C2.1, D1.1 (K), Dsnuber2.1 (K), R6.1, U2.4
- net at U1.13 (OUTCTRL): now also U1.14 (REF), R2.1, R3.2, R7.1, U2.3
- net at U1.15 (2IN-): now also R3.1, R5.2
- net at U1.16 (2IN+): now also R1.1, R2.2
- net at U1.3 (FB): now also R5.1
- net at U1.5 (CT): now also C1.2
- net at U1.6 (RT): now also R4.1
- new net: C5.2, Out2.2 (Pin_2), TR1.7
- new net: Dsnuber2.2 (A), TR1.3
- new net: D3.8 (REF), R10.1, R11.2, R12.1
- new net: C4.1, R10.2
- new net: C3.1, R9.2
- new net: C4.2, C6.2, D3.1 (K), R8.2, U2.2
- new net: C3.2, R8.1, U2.1
Other:
- moved on the sheet: CSnuber1, D2, Q1, RSnuber1, U1

Commit message: Cambios PCB
Parts:
- D3: footprint Package_SO:SOIC-8_3.9x4.9mm_P1.27mm -> Package_TO_SOT_THT:TO-92L
Connections:
- net GND: no longer C6.1, D3.2 (A), D3.3 (A), D3.6 (A), D3.7 (A), R12.2
- net at C5.2, Out2.2 (Pin_2), TR1.7: now also C6.1, D3.2 (A), D3.3 (A), D3.6 (A), D3.7 (A), R12.2
Changed lines of the file:
@@
 $EndComp
 Wire Wire Line
-	8450 1850 8750 1850
+	8450 1850 8700 1850
 Wire Wire Line
 	8600 1750 8600 2450
@@
 F 0 "D3" H 8300 3286 50  0000 C CNN
 F 1 "TL431D" H 8300 3195 50  0000 C CNN
-F 2 "Package_SO:SOIC-8_3.9x4.9mm_P1.27mm" H 8300 3150 50  0001 C CIN
+F 2 "Package_TO_SOT_THT:TO-92L" H 8300 3150 50  0001 C CIN
 F 3 "http://www.ti.com/lit/ds/symlink/tl431.pdf" H 8300 3400 50  0001 C CIN
 	1    8300 3400
@@
 Wire Wire Line
 	8100 2450 8000 2450
-$Comp
-L power:GND #PWR0106
-U 1 1 60FDE657
-P 8600 3400
-F 0 "#PWR0106" H 8600 3150 50  0001 C CNN
-F 1 "GND" H 8605 3227 50  0000 C CNN
-F 2 "" H 8600 3400 50  0001 C CNN
-F 3 "" H 8600 3400 50  0001 C CNN
-	1    8600 3400
-	1    0    0    -1
-$EndComp
 $Comp
 L Device:C C6
@@
 Wire Wire Line
 	8400 3400 8500 3400
-Connection ~ 8600 3400
 Wire Wire Line
 	8200 3400 7700 3400
@@
 Wire Wire Line
 	3350 5050 3350 5950
+Wire Wire Line
+	8700 1850 8700 3400
+Wire Wire Line
+	8700 3400 8600 3400
+Connection ~ 8700 1850
+Wire Wire Line
+	8700 1850 8750 1850
+Connection ~ 8600 3400
 $EndSCHEMATC

Commit message: cambios en PCB
Changed lines of the file:
@@
 EESchema Schematic File Version 4
-LIBS:pcb_flyback-cache
-EELAYER 26 0
+EELAYER 30 0
 EELAYER END
 $Descr A4 11693 8268
@@
 $EndComp
 $Comp
-L Device:R R11
-U 1 1 60FD7C83
-P 8600 2700
-F 0 "R11" H 8670 2746 50  0000 L CNN
-F 1 "R" H 8670 2655 50  0000 L CNN
-F 2 "Resistor_SMD:R_0201_0603Metric" V 8530 2700 50  0001 C CNN
-F 3 "~" H 8600 2700 50  0001 C CNN
-	1    8600 2700
-	1    0    0    -1
-$EndComp
-$Comp
-L Device:R R12
-U 1 1 60FD7D2D
-P 8600 3250
-F 0 "R12" H 8670 3296 50  0000 L CNN
-F 1 "R" H 8670 3205 50  0000 L CNN
-F 2 "Resistor_SMD:R_0201_0603Metric" V 8530 3250 50  0001 C CNN
-F 3 "~" H 8600 3250 50  0001 C CNN
-	1    8600 3250
-	1    0    0    -1
-$EndComp
-$Comp
 L Device:R R10
 U 1 1 60FD7D6F
@@
 	0    1    1    0
 $EndComp
-Wire Wire Line
-	8450 1850 8700 1850
 Wire Wire Line
 	8600 1750 8600 2450
@@
 Connection ~ 8600 2450
 Wire Wire Line
-	8450 2950 8600 2950
-Wire Wire Line
-	8600 2950 8600 2850
-Wire Wire Line
 	8150 2950 8100 2950
 Wire Wire Line
 	7700 2950 7800 2950
-Wire Wire Line
-	8600 3100 8600 3050
-Connection ~ 8600 2950
-Wire Wire Line
-	8300 3300 8300 3050
-Wire Wire Line
-	8300 3050 8600 3050
-Connection ~ 8600 3050
-Wire Wire Line
-	8600 3050 8600 2950
-Wire Wire Line
-	8400 3400 8500 3400
 Wire Wire Line
 	8200 3400 7700 3400
@@
 Wire Wire Line
 	8250 3750 8500 3750
-Wire Wire Line
-	8500 3750 8500 3400
-Connection ~ 8500 3400
-Wire Wire Line
-	8500 3400 8600 3400
 Wire Wire Line
 	7950 3750 7700 3750
@@
 Wire Wire Line
 	3350 5050 3350 5950
+Connection ~ 8600 3400
+Connection ~ 8700 1850
+Wire Wire Line
+	8700 3400 8600 3400
+Wire Wire Line
+	8500 3400 8600 3400
+Wire Wire Line
+	8700 1850 8750 1850
+Wire Wire Line
+	8450 1850 8700 1850
+Wire Wire Line
+	8500 3750 8500 3400
 Wire Wire Line
 	8700 1850 8700 3400
-Wire Wire Line
-	8700 3400 8600 3400
-Connection ~ 8700 1850
-Wire Wire Line
-	8700 1850 8750 1850
-Connection ~ 8600 3400
+Connection ~ 8600 2950
+Wire Wire Line
+	8600 2950 8600 2850
+Wire Wire Line
+	8450 2950 8600 2950
+$Comp
+L Device:R R12
+U 1 1 60FD7D2D
+P 8600 3250
+F 0 "R12" H 8670 3296 50  0000 L CNN
+F 1 "R" H 8670 3205 50  0000 L CNN
+F 2 "Resistor_SMD:R_0201_0603Metric" V 8530 3250 50  0001 C CNN
+F 3 "~" H 8600 3250 50  0001 C CNN
+	1    8600 3250
+	1    0    0    -1
+$EndComp
+$Comp
+L Device:R R11
+U 1 1 60FD7C83
+P 8600 2700
+F 0 "R11" H 8670 2746 50  0000 L CNN
+F 1 "R" H 8670 2655 50  0000 L CNN
+F 2 "Resistor_SMD:R_0201_0603Metric" V 8530 2700 50  0001 C CNN
+F 3 "~" H 8600 2700 50  0001 C CNN
+	1    8600 2700
+	1    0    0    -1
+$EndComp
+Wire Wire Line
+	8600 2950 8600 3050
+Wire Wire Line
+	8300 3300 8300 3050
+Wire Wire Line
+	8300 3050 8600 3050
+Connection ~ 8600 3050
+Wire Wire Line
+	8600 3050 8600 3100
+Wire Wire Line
+	8400 3400 8500 3400
+Connection ~ 8500 3400
 $EndSCHEMATC

Commit message: PCB 99% listo
Parts:
- removed C3: C, Capacitor_SMD:CP_Elec_3x5.3, symbol Device:C
- removed R10, R8: R, Resistor_SMD:R_0201_0603Metric, symbol Device:R
- added Cce1: 1m, Capacitor_SMD:CP_Elec_3x5.3, symbol Device:C
- added Rce1: 8k, Resistor_THT:R_Axial_DIN0204_L3.6mm_D1.6mm_P1.90mm_Vertical, symbol Device:R
- C1: value C -> 1n
- C2, C4: value C -> 22n
- C5: value C -> 500u
- C6: value C -> 1u
- CSnuber1: value C -> 55.2u
- D1: value D_Zener -> 15V
- D2: value DIODE -> RFU10TF6S
- R1, R2: value R -> 51k
- R11: value R -> 38k
- R12, R4: value R -> 10k
- R3: value R -> 510
- R5: value R -> 5.1k
- R6: value R -> 150
- R7: value R -> 860
- R9: value R -> 4.2k
- RSnuber1: value R -> 4k
- TR1: footprint Transformer_SMD:Pulse_PA2777NL -> Transformer_THT:Transformer_Breve_TEZ-28x33
Connections:
- net at C2.1, D1.1 (K), Dsnuber2.1 (K)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: now also Cce1.1
- net at R2.1, R3.2, R7.1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: now also Rce1.2
- net at D3.8 (REF), R11.2, R12.1: now also C4.1
- net at R9.2: now also U2.1
- new net: Cce1.2, Rce1.1
Changed lines of the file:
@@
 EESchema Schematic File Version 4
-EELAYER 30 0
+LIBS:pcb_flyback-cache
+EELAYER 26 0
 EELAYER END
 $Descr A4 11693 8268
@@
 P 5100 2050
 F 0 "RSnuber1" H 5170 2096 50  0000 L CNN
-F 1 "R" H 5170 2005 50  0000 L CNN
+F 1 "4k" H 5170 2005 50  0000 L CNN
 F 2 "Resistor_SMD:R_0201_0603Metric" V 5030 2050 50  0001 C CNN
 F 3 "~" H 5100 2050 50  0001 C CNN
@@
 P 4600 2050
 F 0 "CSnuber1" H 4778 2096 50  0000 L CNN
-F 1 "C" H 4778 2005 50  0000 L CNN
+F 1 "55.2u" H 4778 2005 50  0000 L CNN
 F 2 "Capacitor_SMD:CP_Elec_3x5.3" H 4600 2050 50  0001 C CNN
 F 3 "~" H 4600 2050 50  0001 C CNN
@@
 P 7700 1750
 F 0 "D2" H 7700 1967 50  0000 C CNN
-F 1 "DIODE" H 7700 1876 50  0000 C CNN
+F 1 "RFU10TF6S" H 7700 1876 50  0000 C CNN
 F 2 "Package_TO_SOT_THT:TO-220-2_Vertical" H 7700 1750 50  0001 C CNN
 F 3 "~" H 7700 1750 50  0001 C CNN
@@
 F 0 "TR1" H 6650 2532 50  0000 C CNN
 F 1 "TRANSF6" H 6650 2441 50  0000 C CNN
-F 2 "Transformer_SMD:Pulse_PA2777NL" H 6650 2050 50  0001 C CNN
+F 2 "Transformer_THT:Transformer_Breve_TEZ-28x33" H 6650 2050 50  0001 C CNN
 F 3 "" H 6650 2050 50  0001 C CNN
 	1    6650 2050
@@
 P 6000 3200
 F 0 "C2" H 6115 3246 50  0000 L CNN
-F 1 "C" H 6115 3155 50  0000 L CNN
+F 1 "22n" H 6115 3155 50  0000 L CNN
 F 2 "Capacitor_SMD:CP_Elec_3x5.3" H 6038 3050 50  0001 C CNN
 F 3 "~" H 6000 3200 50  0001 C CNN
@@
 P 4950 3300
 F 0 "D1" V 4904 3379 50  0000 L CNN
-F 1 "D_Zener" V 4995 3379 50  0000 L CNN
+F 1 "15V" V 4995 3379 50  0000 L CNN
 F 2 "Diode_THT:D_DO-35_SOD27_P2.54mm_Vertical_AnodeUp" H 4950 3300 50  0001 C CNN
 F 3 "~" H 4950 3300 50  0001 C CNN
@@
 $EndComp
 $Comp
-L Device:R R10
-U 1 1 60FD7D6F
-P 8300 2950
-F 0 "R10" V 8093 2950 50  0000 C CNN
-F 1 "R" V 8184 2950 50  0000 C CNN
-F 2 "Resistor_SMD:R_0201_0603Metric" V 8230 2950 50  0001 C CNN
-F 3 "~" H 8300 2950 50  0001 C CNN
-	1    8300 2950
-	0    1    1    0
-$EndComp
-$Comp
 L Device:R R9
 U 1 1 60FD7DD0
 P 8250 2450
 F 0 "R9" V 8043 2450 50  0000 C CNN
-F 1 "R" V 8134 2450 50  0000 C CNN
+F 1 "4.2k" V 8134 2450 50  0000 C CNN
 F 2 "Resistor_SMD:R_0201_0603Metric" V 8180 2450 50  0001 C CNN
 F 3 "~" H 8250 2450 50  0001 C CNN
@@
 P 7950 2950
 F 0 "C4" V 7698 2950 50  0000 C CNN
-F 1 "C" V 7789 2950 50  0000 C CNN
+F 1 "22n" V 7789 2950 50  0000 C CNN
 F 2 "Capacitor_SMD:CP_Elec_3x5.3" H 7988 2800 50  0001 C CNN
 F 3 "~" H 7950 2950 50  0001 C CNN
 	1    7950 2950
-	0    1    1    0
-$EndComp
-$Comp
-L Device:C C3
-U 1 1 60FDAE93
-P 7850 2450
-F 0 "C3" V 7598 2450 50  0000 C CNN
-F 1 "C" V 7689 2450 50  0000 C CNN
-F 2 "Capacitor_SMD:CP_Elec_3x5.3" H 7888 2300 50  0001 C CNN
-F 3 "~" H 7850 2450 50  0001 C CNN
-	1    7850 2450
 	0    1    1    0
 $EndComp
@@
 	-1   0    0    -1
 $EndComp
-Wire Wire Line
-	8100 2450 8000 2450
 $Comp
 L Device:C C6
@@
 P 8100 3750
 F 0 "C6" V 7848 3750 50  0000 C CNN
-F 1 "C" V 7939 3750 50  0000 C CNN
+F 1 "1u" V 7939 3750 50  0000 C CNN
 F 2 "Capacitor_SMD:CP_Elec_3x5.3" H 8138 3600 50  0001 C CNN
 F 3 "~" H 8100 3750 50  0001 C CNN
 	1    8100 3750
 	0    1    1    0
-$EndComp
-$Comp
-L Device:R R8
-U 1 1 60FE2CEB
-P 7450 2850
-F 0 "R8" H 7520 2896 50  0000 L CNN
-F 1 "R" H 7520 2805 50  0000 L CNN
-F 2 "Resistor_SMD:R_0201_0603Metric" V 7380 2850 50  0001 C CNN
-F 3 "~" H 7450 2850 50  0001 C CNN
-	1    7450 2850
-	1    0    0    -1
 $EndComp
 $Comp
@@
 P 6650 3200
 F 0 "R7" H 6720 3246 50  0000 L CNN
-F 1 "R" H 6720 3155 50  0000 L CNN
+F 1 "860" H 6720 3155 50  0000 L CNN
 F 2 "Resistor_SMD:R_0201_0603Metric" V 6580 3200 50  0001 C CNN
 F 3 "~" H 6650 3200 50  0001 C CNN
@@
 P 3100 5050
 F 0 "R2" V 2893 5050 50  0000 C CNN
-F 1 "R" V 2984 5050 50  0000 C CNN
+F 1 "51k" V 2984 5050 50  0000 C CNN
 F 2 "Resistor_SMD:R_0201_0603Metric" V 3030 5050 50  0001 C CNN
 F 3 "~" H 3100 5050 50  0001 C CNN
@@
 P 2650 5050
 F 0 "R1" V 2443 5050 50  0000 C CNN
-F 1 "R" V 2534 5050 50  0000 C CNN
+F 1 "51k" V 2534 5050 50  0000 C CNN
 F 2 "Resistor_SMD:R_0201_0603Metric" V 2580 5050 50  0001 C CNN
 F 3 "~" H 2650 5050 50  0001 C CNN
@@
 P 3800 5350
 F 0 "R4" V 3593 5350 50  0000 C CNN
-F 1 "R" V 3684 5350 50  0000 C CNN
+F 1 "10k" V 3684 5350 50  0000 C CNN
 F 2 "Resistor_SMD:R_0201_0603Metric" V 3730 5350 50  0001 C CNN
 F 3 "~" H 3800 5350 50  0001 C CNN
@@
 P 5100 4050
 F 0 "R6" V 5307 4050 50  0000 C CNN
-F 1 "R" V 5216 4050 50  0000 C CNN
+F 1 "150" V 5216 4050 50  0000 C CNN
 F 2 "Resistor_SMD:R_0201_0603Metric" V 5030 4050 50  0001 C CNN
 F 3 "~" H 5100 4050 50  0001 C CNN
@@
 P 8100 1950
 F 0 "C5" H 8215 1996 50  0000 L CNN
-F 1 "C" H 8215 1905 50  0000 L CNN
+F 1 "500u" H 8215 1905 50  0000 L CNN
 F 2 "Capacitor_SMD:CP_Elec_3x5.3" H 8138 1800 50  0001 C CNN
 F 3 "~" H 8100 1950 50  0001 C CNN
@@
 Connection ~ 8600 2450
 Wire Wire Line
-	8150 2950 8100 2950
-Wire Wire Line
 	7700 2950 7800 2950
 Wire Wire Line
@@
 	7700 2950 7700 3400
 Wire Wire Line
-	7700 3400 7450 3400
-Wire Wire Line
 	7250 3400 7250 2950
 Wire Wire Line
 	7250 2750 7250 2450
 Wire Wire Line
-	7250 2450 7450 2450
-Wire Wire Line
-	7450 3000 7450 3400
-Connection ~ 7450 3400
-Wire Wire Line
-	7450 3400 7250 3400
-Wire Wire Line
-	7450 2700 7450 2450
-Connection ~ 7450 2450
-Wire Wire Line
-	7450 2450 7700 2450
-Wire Wire Line
-	6650 2750 6150 2750
+	6650 2750 6250 2750
 Wire Wire Line
 	6150 2750 6150 3000
@@
 P 3750 4750
 F 0 "R3" V 3543 4750 50  0000 C CNN
-F 1 "R" V 3634 4750 50  0000 C CNN
+F 1 "510" V 3634 4750 50  0000 C CNN
 F 2 "Resistor_SMD:R_0201_0603Metric" V 3680 4750 50  0001 C CNN
 F 3 "~" H 3750 4750 50  0001 C CNN
@@
 P 4050 4950
 F 0 "R5" V 3843 4950 50  0000 C CNN
-F 1 "R" V 3934 4950 50  0000 C CNN
+F 1 "5.1k" V 3934 4950 50  0000 C CNN
 F 2 "Resistor_SMD:R_0201_0603Metric" V 3980 4950 50  0001 C CNN
 F 3 "~" H 4050 4950 50  0001 C CNN
@@
 P 3800 5700
 F 0 "C1" V 4052 5700 50  0000 C CNN
-F 1 "C" V 3961 5700 50  0000 C CNN
+F 1 "1n" V 3961 5700 50  0000 C CNN
 F 2 "Capacitor_SMD:CP_Elec_3x5.3" H 3838 5550 50  0001 C CNN
 F 3 "~" H 3800 5700 50  0001 C CNN
@@
 $EndComp
 Wire Wire Line
-	6650 2950 6400 2950
-Wire Wire Line
-	6400 2950 6400 5950
-Connection ~ 6650 2950
-Wire Wire Line
 	5400 4050 5250 4050
 Wire Wire Line
@@
 Wire Wire Line
 	8600 2950 8600 2850
-Wire Wire Line
-	8450 2950 8600 2950
 $Comp
 L Device:R R12
@@
 P 8600 3250
 F 0 "R12" H 8670 3296 50  0000 L CNN
-F 1 "R" H 8670 3205 50  0000 L CNN
+F 1 "10k" H 8670 3205 50  0000 L CNN
 F 2 "Resistor_SMD:R_0201_0603Metric" V 8530 3250 50  0001 C CNN
 F 3 "~" H 8600 3250 50  0001 C CNN
@@
 P 8600 2700
 F 0 "R11" H 8670 2746 50  0000 L CNN
-F 1 "R" H 8670 2655 50  0000 L CNN
+F 1 "38k" H 8670 2655 50  0000 L CNN
 F 2 "Resistor_SMD:R_0201_0603Metric" V 8530 2700 50  0001 C CNN
 F 3 "~" H 8600 2700 50  0001 C CNN
@@
 	8400 3400 8500 3400
 Connection ~ 8500 3400
+Wire Wire Line
+	7250 3400 7700 3400
+Wire Wire Line
+	7250 2450 8100 2450
+$Comp
+L Device:C Cce1
+U 1 1 6103A31D
+P 6250 3600
+F 0 "Cce1" H 6365 3646 50  0000 L CNN
+F 1 "1m" H 6365 3555 50  0000 L CNN
+F 2 "Capacitor_SMD:CP_Elec_3x5.3" H 6288 3450 50  0001 C CNN
+F 3 "~" H 6250 3600 50  0001 C CNN
+	1    6250 3600
+	1    0    0    -1
+$EndComp
+$Comp
+L Device:R Rce1
+U 1 1 6103A40A
+P 6250 3900
+F 0 "Rce1" H 6320 3946 50  0000 L CNN
+F 1 "8k" H 6320 3855 50  0000 L CNN
+F 2 "Resistor_THT:R_Axial_DIN0204_L3.6mm_D1.6mm_P1.90mm_Vertical" V 6180 3900 50  0001 C CNN
+F 3 "~" H 6250 3900 50  0001 C CNN
+	1    6250 3900
+	1    0    0    -1
+$EndComp
+Wire Wire Line
+	6250 3450 6250 2750
+Connection ~ 6250 2750
+Wire Wire Line
+	6250 2750 6150 2750
+Wire Wire Line
+	6250 4050 6250 4100
+Wire Wire Line
+	6250 4100 6400 4100
+Wire Wire Line
+	6400 4100 6400 5950
+Wire Wire Line
+	6650 2950 6550 2950
+Wire Wire Line
+	6550 2950 6550 4100
+Wire Wire Line
+	6550 4100 6400 4100
+Connection ~ 6650 2950
+Connection ~ 6400 4100
+Wire Wire Line
+	8100 2950 8600 2950
 $EndSCHEMATC
