File: PCB/pcb_flyback/pcb_flyback.kicad_pcb (KiCad board)
At the start: 2 copper layers, 31 parts, among them Q1 IRF540N, U1 TL494, U2 PC817

Commit message: cambios en PCB
Parts:
- U2: moved to F.Cu
- moved C6 29.9 mm to (116.8, 106.7), turned to 90 degrees
- moved R8 21.9 mm to (114.3, 113.0), turned to 0 degrees
- moved U2 21.6 mm to (116.8, 116.8), turned to 270 degrees
- moved Dsnuber2 20.4 mm to (123.2, 116.8), turned to 90 degrees
- moved R3 14.9 mm to (95.2, 114.3), turned to 90 degrees
- moved R2 14.0 mm to (90.2, 114.3), turned to 270 degrees
- moved R5 9.67 mm to (100.3, 124.5), turned to 90 degrees
- moved R1 6.84 mm to (85.1, 114.3)
- moved R7 4.58 mm to (105.4, 124.5), turned to 90 degrees
- moved C1 2.62 mm to (111.8, 106.7), turned to 90 degrees
- moved R4 2.54 mm to (114.3, 101.6)
Routing:
- net Net-(R5-Pad1): track 20.4 -> 45.8 mm
- net Net-(C2-Pad1): track 34.0 -> 54.1 mm
- net Net-(C4-Pad2): track 56.9 -> 44.2 mm
- net GND: track 163.6 -> 151.9 mm
- net Net-(R2-Pad1): track 52.1 -> 42.8 mm
- net Net-(C3-Pad2): track 37.0 -> 27.7 mm
- net Net-(R1-Pad1): track 24.8 -> 16.7 mm
- net Net-(Dsnuber2-Pad2): track 16.8 -> 24.0 mm
- net Net-(R3-Pad1): track 17.8 -> 14.6 mm
- net Net-(R4-Pad1): track 4.26 -> 5.31 mm
- net Net-(C1-Pad2): track 4.37 -> 5.33 mm

Commit message: cambios en los bancos de prueba de fuente y controlador
Parts:
- D3: footprint Package_SO:SOIC-8_3.9x4.9mm_P1.27mm -> Package_TO_SOT_THT:TO-92
- RSnuber1: footprint Resistor_SMD:R_0805_2012Metric -> Resistor_THT:R_Axial_DIN0207_L6.3mm_D2.5mm_P10.16mm_Horizontal
- TR1: footprint Transformer_SMD:Pulse_PA2777NL -> Transformer_THT:Transformer_Breve_TEZ-22x24
- U1: footprint Package_DIP:DIP-16_W7.62mm_SMDSocket_SmallPads -> Package_DIP:DIP-16_W7.62mm
- moved R8 25.6 mm to (91.4, 124.5), turned to 270 degrees
- moved R9 25.0 mm to (121.9, 124.5)
- moved R7 22.9 mm to (92.7, 105.4)
- moved U2 22.9 mm to (95.2, 124.5), turned to 0 degrees
- moved C3 20.7 mm to (108.0, 118.1)
- moved R11 19.4 mm to (129.5, 120.7), turned to 90 degrees
- moved RSnuber1 18.2 mm to (91.4, 86.4), turned to 0 degrees
- moved Dsnuber2 18.2 mm to (106.7, 124.5), turned to 0 degrees
- moved R10 17.6 mm to (121.9, 118.1)
- moved CSnuber1 17.3 mm to (86.4, 87.6)
- moved Out1 16.5 mm to (82.5, 86.4), turned to 180 degrees
- moved C4 15.5 mm to (115.6, 118.1)
- moved Out2 15.3 mm to (141.0, 102.9), turned to 270 degrees
- moved C5 15.2 mm to (138.4, 113.0)
- moved Dsnuber1 14.1 mm to (91.4, 90.2)
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Routing:
- net Net-(R5-Pad1): track 45.8 -> 11.6 mm
- net Net-(Dsnuber2-Pad2): track 24.0 -> 0.00 mm
- net GND: track 151.9 -> 138.1 mm
- net Net-(C3-Pad2): track 27.7 -> 18.3 mm
- net Net-(C5-Pad2): track 13.7 -> 22.4 mm
- net Net-(C5-Pad1): track 32.8 -> 41.2 mm
- net Net-(C3-Pad1): track 6.56 -> 14.6 mm
- net Net-(D3-Pad8): track 18.9 -> 10.9 mm
- net Net-(CSnuber1-Pad2): track 9.42 -> 17.2 mm
- net Net-(Dsnuber1-Pad2): track 14.3 -> 21.1 mm
- net Net-(CSnuber1-Pad1): track 32.1 -> 38.6 mm
- net Net-(R3-Pad1): track 14.6 -> 21.0 mm
- net Net-(R2-Pad1): track 42.8 -> 37.7 mm
- net Net-(C2-Pad1): track 54.1 -> 50.8 mm
- net Net-(C4-Pad1): track 5.05 -> 3.36 mm
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- added copper zone on B.Cu, net GND

Commit message: Cambios PCB, faltan otros
Parts:
- Out2: footprint Connector_PinHeader_1.00mm:PinHeader_1x02_P1.00mm_Vertical -> Connector_Wire:SolderWirePad_1x02_P3.81mm_Drill0.8mm
Connections:
- C6 pad 1: GND -> Net-(C5-Pad2)
- D3 pad 2: GND -> Net-(C5-Pad2)
- D3 pad 3: GND -> Net-(C5-Pad2)
- R12 pad 2: GND -> Net-(C5-Pad2)
Routing:
- net Net-(C5-Pad2): track 22.4 -> 45.5 mm
- net GND: track 138.1 -> 133.4 mm
- net Net-(C5-Pad1): track 41.2 -> 44.0 mm
Changed lines of the file:
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@@
     (thickness 1.6)
     (drawings 6)
-    (tracks 150)
+    (tracks 155)
     (zones 0)
     (modules 31)
@@
     (add_net "Net-(U1-Pad9)")
   )
+  (module Connector_Wire:SolderWirePad_1x02_P3.81mm_Drill0.8mm (layer F.Cu)
+    (at 140.97 102.87 270)
+    (descr "Wire solder connection")
+    (tags connector)
+    (attr virtual)
+    (fp_text reference Out2 (at 1.905 -2.5 270) (layer F.SilkS)
+      (effects (font (size 1 1) (thickness 0.15)))
+    )
+    (fp_text value Screw_Terminal_01x02 (at 1.905 2.54 270) (layer F.Fab)
+      (effects (font (size 1 1) (thickness 0.15)))
+    )
+    (fp_line (start 5.31 1.5) (end -1.49 1.5) (layer F.CrtYd) (width 0.05))
+    (fp_line (start 5.31 1.5) (end 5.31 -1.5) (layer F.CrtYd) (width 0.05))
+    (fp_line (start -1.49 -1.5) (end -1.49 1.5) (layer F.CrtYd) (width 0.05))
+    (fp_line (start -1.49 -1.5) (end 5.31 -1.5) (layer F.CrtYd) (width 0.05))
+    (fp_text user %R (at 1.905 0 270) (layer F.Fab)
+      (effects (font (size 1 1) (thickness 0.15)))
+    )
+    (pad 2 thru_hole circle (at 3.81 0 270) (size 1.99898 1.99898) (drill 0.8001) (layers *.Cu *.Mask)
+      (net 8 "Net-(C5-Pad2)"))
+    (pad 1 thru_hole rect (at 0 0 270) (size 1.99898 1.99898) (drill 0.8001) (layers *.Cu *.Mask)
+      (net 9 "Net-(C5-Pad1)"))
+  )
   (module Package_DIP:DIP-16_W7.62mm (layer F.Cu)
     (at 105.41 113.03 180)
@@
       (net 7 "Net-(C4-Pad2)"))
     (pad 3 thru_hole circle (at 2.54 0 90) (size 1.3 1.3) (drill 0.75) (layers *.Cu *.Mask)
-      (net 1 GND))
+      (net 8 "Net-(C5-Pad2)"))
     (pad 2 thru_hole circle (at 1.27 -1.27 90) (size 1.3 1.3) (drill 0.75) (layers *.Cu *.Mask)
-      (net 1 GND))
+      (net 8 "Net-(C5-Pad2)"))
     (model ${KISYS3DMOD}/Package_TO_SOT_THT.3dshapes/TO-92.wrl
       (at (xyz 0 0 0))
@@
       (net 10 "Net-(CSnuber1-Pad1)"))
     (model ${KISYS3DMOD}/Resistor_THT.3dshapes/R_Axial_DIN0207_L6.3mm_D2.5mm_P10.16mm_Horizontal.wrl
-      (at (xyz 0 0 0))
-      (scale (xyz 1 1 1))
-      (rotate (xyz 0 0 0))
-    )
-  )
-  (module Connector_PinHeader_1.00mm:PinHeader_1x02_P1.00mm_Vertical (layer F.Cu)
-    (at 140.97 102.87 270)
-    (descr "Through hole straight pin header, 1x02, 1.00mm pitch, single row")
-    (tags "Through hole pin header THT 1x02 1.00mm single row")
-    (fp_text reference Out2 (at 0 -1.56 270) (layer F.SilkS)
-      (effects (font (size 1 1) (thickness 0.15)))
-    )
-    (fp_text value Screw_Terminal_01x02 (at 0 2.56 270) (layer F.Fab)
-      (effects (font (size 1 1) (thickness 0.15)))
-    )
-    (fp_text user %R (at 0 0.5) (layer F.Fab)
-      (effects (font (size 0.76 0.76) (thickness 0.114)))
-    )
-    (fp_line (start 1.15 -1) (end -1.15 -1) (layer F.CrtYd) (width 0.05))
-    (fp_line (start 1.15 2) (end 1.15 -1) (layer F.CrtYd) (width 0.05))
-    (fp_line (start -1.15 2) (end 1.15 2) (layer F.CrtYd) (width 0.05))
-    (fp_line (start -1.15 -1) (end -1.15 2) (layer F.CrtYd) (width 0.05))
-    (fp_line (start -0.695 -0.685) (end 0 -0.685) (layer F.SilkS) (width 0.12))
-    (fp_line (start -0.695 0) (end -0.695 -0.685) (layer F.SilkS) (width 0.12))
-    (fp_line (start 0.608276 0.685) (end 0.695 0.685) (layer F.SilkS) (width 0.12))
-    (fp_line (start -0.695 0.685) (end -0.608276 0.685) (layer F.SilkS) (width 0.12))
-    (fp_line (start 0.695 0.685) (end 0.695 1.56) (layer F.SilkS) (width 0.12))
-    (fp_line (start -0.695 0.685) (end -0.695 1.56) (layer F.SilkS) (width 0.12))
-    (fp_line (start 0.394493 1.56) (end 0.695 1.56) (layer F.SilkS) (width 0.12))
-    (fp_line (start -0.695 1.56) (end -0.394493 1.56) (layer F.SilkS) (width 0.12))
-    (fp_line (start -0.635 -0.1825) (end -0.3175 -0.5) (layer F.Fab) (width 0.1))
-    (fp_line (start -0.635 1.5) (end -0.635 -0.1825) (layer F.Fab) (width 0.1))
-    (fp_line (start 0.635 1.5) (end -0.635 1.5) (layer F.Fab) (width 0.1))
-    (fp_line (start 0.635 -0.5) (end 0.635 1.5) (layer F.Fab) (width 0.1))
-    (fp_line (start -0.3175 -0.5) (end 0.635 -0.5) (layer F.Fab) (width 0.1))
-    (pad 2 thru_hole oval (at 0 1 270) (size 0.85 0.85) (drill 0.5) (layers *.Cu *.Mask)
-      (net 8 "Net-(C5-Pad2)"))
-    (pad 1 thru_hole rect (at 0 0 270) (size 0.85 0.85) (drill 0.5) (layers *.Cu *.Mask)
-      (net 9 "Net-(C5-Pad1)"))
-    (model ${KISYS3DMOD}/Connector_PinHeader_1.00mm.3dshapes/PinHeader_1x02_P1.00mm_Vertical.wrl
       (at (xyz 0 0 0))
       (scale (xyz 1 1 1))
@@
     )
     (pad 1 smd rect (at -1.5 0 270) (size 2.2 1.6) (layers F.Cu F.Paste F.Mask)
-      (net 1 GND))
+      (net 8 "Net-(C5-Pad2)"))
     (pad 2 smd rect (at 1.5 0 270) (size 2.2 1.6) (layers F.Cu F.Paste F.Mask)
       (net 7 "Net-(C4-Pad2)"))
@@
     (fp_line (start -3.15 1.6) (end -3.15 -1.6) (layer F.Fab) (width 0.1))
     (pad 2 smd roundrect (at 2.9875 0 180) (size 1.525 3.35) (layers F.Cu F.Paste F.Mask) (roundrect_rratio 0.163934)
-      (net 1 GND))
+      (net 8 "Net-(C5-Pad2)"))
     (pad 1 smd roundrect (at -2.9875 0 180) (size 1.525 3.35) (layers F.Cu F.Paste F.Mask) (roundrect_rratio 0.163934)
       (net 13 "Net-(D3-Pad8)"))
@@
   (segment (start 110.49 96.0725) (end 110.49 92.71) (width 0.25) (layer F.Cu) (net 1) (status 400000))
   (segment (start 110.49 92.71) (end 109.22 91.44) (width 0.25) (layer F.Cu) (net 1) (status 800000))
-  (segment (start 119.38 111.76) (end 124.0125 111.76) (width 0.25) (layer F.Cu) (net 1) (status C00000))
   (segment (start 101.6 106.68) (end 104.14 106.68) (width 0.25) (layer B.Cu) (net 1))
   (segment (start 104.14 106.68) (end 105.41 105.41) (width 0.25) (layer B.Cu) (net 1) (status 800000))
@@
   (segment (start 91.44 127.4475) (end 94.8025 127.4475) (width 0.25) (layer F.Cu) (net 7) (status C00000))
   (segment (start 94.8025 127.4475) (end 95.25 127) (width 0.25) (layer F.Cu) (net 7) (status C00000))
-  (segment (start 139.97 102.87) (end 139.97 109.99) (width 0.25) (layer F.Cu) (net 8) (status 400000))
-  (segment (start 139.97 109.99) (end 138.43 111.53) (width 0.25) (layer F.Cu) (net 8) (status 800000))
-  (segment (start 133.11 92.63) (end 133.11 93.74) (width 0.25) (layer F.Cu) (net 8) (status 400000))
-  (segment (start 139.97 100.6) (end 139.97 102.87) (width 0.25) (layer F.Cu) (net 8) (status 800000))
-  (segment (start 133.11 93.74) (end 139.97 100.6) (width 0.25) (layer F.Cu) (net 8))
+  (segment (start 138.43 111.53) (end 138.43 109.22) (width 0.25) (layer F.Cu) (net 8) (status 400000))
+  (segment (start 138.43 109.22) (end 140.97 106.68) (width 0.25) (layer F.Cu) (net 8) (status 800000))
+  (segment (start 140.97 106.68) (end 139.7 106.68) (width 0.25) (layer F.Cu) (net 8) (status 400000))
+  (segment (start 138.43 97.95) (end 133.11 92.63) (width 0.25) (layer F.Cu) (net 8) (status 800000))
+  (segment (start 138.43 105.41) (end 138.43 97.95) (width 0.25) (layer F.Cu) (net 8))
+  (segment (start 139.7 106.68) (end 138.43 105.41) (width 0.25) (layer F.Cu) (net 8))
+  (segment (start 124.0125 111.76) (end 124.0125 110.9375) (width 0.25) (layer F.Cu) (net 8) (status C00000))
+  (segment (start 136.12 109.22) (end 138.43 111.53) (width 0.25) (layer F.Cu) (net 8) (status 800000))
+  (segment (start 125.73 109.22) (end 136.12 109.22) (width 0.25) (layer F.Cu) (net 8))
+  (segment (start 124.0125 110.9375) (end 125.73 109.22) (width 0.25) (layer F.Cu) (net 8) (status 400000))
+  (segment (start 119.38 111.76) (end 124.0125 111.76) (width 0.25) (layer F.Cu) (net 8) (status C00000))
   (segment (start 124.9075 124.46) (end 128.7175 124.46) (width 0.25) (layer F.Cu) (net 9) (status 400000))
   (segment (start 128.7175 124.46) (end 129.54 123.6375) (width 0.25) (layer F.Cu) (net 9) (status 800000))
   (segment (start 129.54 123.6375) (end 129.54 123.42) (width 0.25) (layer F.Cu) (net 9) (status C00000))
   (segment (start 129.54 123.42) (end 138.43 114.53) (width 0.25) (layer F.Cu) (net 9) (status C00000))
-  (segment (start 138.43 114.53) (end 138.43 114.3) (width 0.25) (layer F.Cu) (net 9) (status C00000))
-  (segment (start 140.97 111.76) (end 140.97 102.87) (width 0.25) (layer F.Cu) (net 9) (status 800000))
-  (segment (start 138.43 114.3) (end 140.97 111.76) (width 0.25) (layer F.Cu) (net 9) (status 400000))
-  (segment (start 139.7 92.71) (end 139.7 99.06) (width 0.25) (layer F.Cu) (net 9) (status 400000))
-  (segment (start 140.97 100.33) (end 140.97 102.87) (width 0.25) (layer F.Cu) (net 9) (status 800000))
-  (segment (start 139.7 99.06) (end 140.97 100.33) (width 0.25) (layer F.Cu) (net 9))
+  (segment (start 139.7 92.71) (end 139.7 101.6) (width 0.25) (layer F.Cu) (net 9) (status 400000))
+  (segment (start 139.7 101.6) (end 140.97 102.87) (width 0.25) (layer F.Cu) (net 9) (status 800000))
+  (segment (start 140.97 102.87) (end 142.24 102.87) (width 0.25) (layer F.Cu) (net 9) (status 400000))
+  (segment (start 143.51 109.45) (end 138.43 114.53) (width 0.25) (layer F.Cu) (net 9) (status 800000))
+  (segment (start 143.51 104.14) (end 143.51 109.45) (width 0.25) (layer F.Cu) (net 9))
+  (segment (start 142.24 102.87) (end 143.51 104.14) (width 0.25) (layer F.Cu) (net 9))
   (segment (start 82.55 85.36) (end 85.59 85.36) (width 0.25) (layer F.Cu) (net 10) (status C00000))
   (segment (start 85.59 85.36) (end 86.59 86.36) (width 0.25) (layer F.Cu) (net 10) (status C00000))

Commit message: Cambios PCB
Parts:
- D3: footprint Package_TO_SOT_THT:TO-92 -> Package_TO_SOT_THT:TO-92L
- moved D3 2.54 mm to (119.4, 111.8), turned to 180 degrees
Routing:
- net GND: track 133.4 -> 111.1 mm
- net Net-(C4-Pad2): track 43.4 -> 35.9 mm
- net Net-(C5-Pad2): track 45.5 -> 40.9 mm

Commit message: cambios en PCB
Parts:
- removed D3: TL431D, Package_TO_SOT_THT:TO-92L
- added REF** (x3): TO-92L_Wide, Package_TO_SOT_THT:TO-92L_Wide, F.Cu at (0.00, 0.00)
- added REF** (x6): TO-92, Package_TO_SOT_THT:TO-92, F.Cu at (0.00, 0.00)
- added REF** (x4): TO-92L, Package_TO_SOT_THT:TO-92L, F.Cu at (0.00, 0.00)
- turned C6 to 90 degrees
Routing:
- net Net-(C5-Pad2): track 40.9 -> 58.6 mm
- net Net-(C4-Pad2): track 35.9 -> 52.3 mm
- net GND: track 111.1 -> 107.6 mm

Commit message: PCB 99% listo
Parts:
- removed C3: C, Capacitor_THT:CP_Radial_Tantal_D4.5mm_P2.50mm
- removed R8: R, Resistor_SMD:R_2512_6332Metric_Pad1.52x3.35mm_HandSolder
- removed REF** (x3): TO-92L_Wide, Package_TO_SOT_THT:TO-92L_Wide
- removed REF** (x6): TO-92, Package_TO_SOT_THT:TO-92
- removed REF** (x4): TO-92L, Package_TO_SOT_THT:TO-92L
- added Cce1: 1m, Capacitor_SMD:CP_Elec_3x5.3, F.Cu at (86.4, 125.7)
- added D3: TL431D, Package_TO_SOT_THT:TO-92L, F.Cu at (115.6, 119.4)
- added Rce1: 8k, Resistor_THT:R_Axial_DIN0204_L3.6mm_D1.6mm_P1.90mm_Vertical, F.Cu at (90.2, 125.7)
- C1: value C -> 1n
- C2, C4: value C -> 22n
- C5: value C -> 500u
- C6: value C -> 1u
- CSnuber1: value C -> 55.2u
- D1: value D_Zener -> 15V
- D2: value DIODE -> RFU10TF6S
- R1, R2: value R -> 51k
- R10: value R -> 1m
- R11: value R -> 38k
- R12, R4: value R -> 10k
- R3: value R -> 510
- R5: value R -> 5.1k
- R6: value R -> 150
- R7: value R -> 860
- R9: value R -> 4.2k; footprint Resistor_SMD:R_2512_6332Metric_Pad1.52x3.35mm_HandSolder -> Resistor_SMD:R_1206_3216Metric
- RSnuber1: value R -> 4k
- TR1: footprint Transformer_THT:Transformer_Breve_TEZ-22x24 -> Transformer_THT:Transformer_Breve_TEZ-28x33
- moved R9 8.13 mm to (115.6, 129.5)
- moved D2 7.62 mm to (147.3, 87.6)
- moved R12 7.62 mm to (127.0, 119.4)
- moved C4 6.48 mm to (114.3, 124.5)
- moved R10 6.48 mm to (120.7, 124.5)
- moved U2 6.35 mm to (95.2, 130.8), turned to 90 degrees
- moved Out2 6.35 mm to (147.3, 102.9)
- moved C5 4.58 mm to (135.9, 116.8)
- moved R11 3.81 mm to (129.5, 124.5), turned to 180 degrees
- turned C6 to 270 degrees
- turned Dsnuber2 to 90 degrees
Connections:
- R11 pad 2: Net-(D3-Pad8) -> Net-(C4-Pad1)
- R12 pad 1: Net-(D3-Pad8) -> Net-(C4-Pad1)
- R9 pad 2: Net-(C3-Pad1) -> Net-(R9-Pad2)
- U2 pad 1: Net-(C3-Pad2) -> Net-(R9-Pad2)
Routing:
- net Net-(C4-Pad2): track 52.3 -> 31.7 mm
- net Net-(R9-Pad2): track 0.00 -> 20.5 mm
- net Net-(C2-Pad1): track 50.8 -> 70.9 mm
- net Net-(C4-Pad1): track 3.36 -> 23.4 mm
- net Net-(C3-Pad2): track 18.3 -> 0.00 mm
- net Net-(C5-Pad1): track 44.0 -> 60.5 mm
- net Net-(Dsnuber2-Pad2): track 0.00 -> 15.2 mm
- net Net-(C3-Pad1): track 14.6 -> 0.00 mm
- net Net-(D3-Pad8): track 10.9 -> 0.00 mm
- net Net-(D2-Pad1): track 6.59 -> 13.8 mm
- net GND: track 107.6 -> 101.6 mm
- net Net-(Cce1-Pad2): track 0.00 -> 4.43 mm
- net Net-(R2-Pad1): track 37.7 -> 41.2 mm
- net Net-(C5-Pad2): track 58.6 -> 59.7 mm
Other:
- net class Default: trace_width 0.25 -> 0.6

Commit message: PCB 99,9% listo
Routing:
- net GND: track 101.6 -> 107.6 mm
Changed lines of the file:
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@@
     (thickness 1.6)
     (drawings 1)
-    (tracks 163)
+    (tracks 166)
     (zones 0)
     (modules 31)
@@
   (segment (start 93.98 104.14) (end 93.98 92.71) (width 0.25) (layer B.Cu) (net 1))
   (segment (start 91.44 106.68) (end 93.98 104.14) (width 0.25) (layer B.Cu) (net 1))
+  (segment (start 105.41 110.49) (end 107.95 110.49) (width 0.6) (layer F.Cu) (net 1) (status 400000))
+  (segment (start 110.26 108.18) (end 110.49 108.18) (width 0.6) (layer F.Cu) (net 1) (status C00000))
+  (segment (start 107.95 110.49) (end 110.26 108.18) (width 0.6) (layer F.Cu) (net 1) (status 800000))
   (segment (start 105.41 102.87) (end 106.68 102.87) (width 0.25) (layer F.Cu) (net 2) (status 400000))
   (segment (start 108.99 105.18) (end 110.49 105.18) (width 0.25) (layer F.Cu) (net 2) (status 800000))
